File: RS-485_interface.kicad_sch (KiCad schematic)
At the start: 5 parts, among them J4 Screw_Terminal_01x03, U3 ADM3483ARZ

Commit message: version 1
Parts:
- J2: renamed from J4; footprint (none) -> Library:CUI_TB007-508-03BE
- R2: renamed from R5; value R_US -> 1k; footprint (none) -> Resistor_SMD:R_0805_2012Metric_Pad1.20x1.40mm_HandSolder
- R3: renamed from R6; value R_US -> 1k; footprint (none) -> Resistor_SMD:R_0805_2012Metric_Pad1.20x1.40mm_HandSolder
- R4: renamed from R7; value R_US -> 120; footprint (none) -> Resistor_THT:R_Axial_DIN0207_L6.3mm_D2.5mm_P7.62mm_Horizontal
- U2: renamed from U3; footprint R_8_ADI -> Library:R_8_ADI
Connections:
- net RS-485 RX enable renamed ~{RS-485 RX enable}
Other:
- company: (none) -> Texas A&M ECEN Capstone
- title: (none) -> RS-485 Interface
- moved on the sheet: R2, R3
