File: power_and_usb.kicad_sch (KiCad schematic)
At the start: 28 parts, among them J5 USB4105GFA, Q1 SS8050-G, Q2 SS8050-G, U6 LM2595S-5, U7 LM2595S-3.3, U8 CP2102N-A02-GQFN24R

Commit message: unknown latest changes
Parts:
- removed R?: 47.5kΩ, Resistor_SMD:R_0805_2012Metric_Pad1.20x1.40mm_HandSolder, symbol Device:R_US
- removed R?: 22.1kΩ, Resistor_SMD:R_0805_2012Metric_Pad1.20x1.40mm_HandSolder, symbol Device:R_US
- gave numbers to parts that had none: 9
Connections:
- net +5V: no longer C28.1, U7.2 (VIN)
- net VBUS: now also U8.8 (VBUS)
- new net: C28.1, U7.2 (VIN)
